Commit message: FIXED BUG

File: robots/descriptions/go2_description/xacro/leg.xacro (robot description, xacro)
@@ -155,5 +155,5 @@
             </inertial>
         </link>
-        <ros2_control name="${name}" type="system">
+        <!-- <ros2_control name="${name}" type="system">
             <hardware>
                 <plugin>gazebo_ros2_control/GazeboSystem</plugin>
@@ -174,5 +174,5 @@
                 <state_interface name="velocity"/>
             </joint>
-        </ros2_control>
+        </ros2_control>  -->
         <!-- <xacro:leg_transmission name="${name}"/> -->
     </xacro:macro>

File: robots/descriptions/go2_description/xacro/robot_mid360_depth_camera.xacro (robot description, xacro)
@@ -97,3 +97,72 @@
         <origin xyz="0.23 0 0.07" rpy="0 0 0"/>
     </xacro:depth_camera>
+    <ros2_control name="go2_hardware" type="system">
+        <hardware>
+            <plugin>gazebo_ros2_control/GazeboSystem</plugin>
+            <!-- This param points to the ros_control configuration YAML. -->
+            <!-- It's crucial for the plugin to know which controllers to manage. -->
+            <param name="ros_control_config_file">$(find go2_description)/config/ros_control/ros_control.yaml</param>
+        </hardware>
+        <!-- Define ALL 12 robot joints here -->
+        <joint name="lf_hip_joint">
+            <command_interface name="effort"/>
+            <state_interface name="position"/>
+            <state_interface name="velocity"/>
+        </joint>
+        <joint name="lf_upper_leg_joint">
+            <command_interface name="effort"/>
+            <state_interface name="position"/>
+            <state_interface name="velocity"/>
+        </joint>
+        <joint name="lf_lower_leg_joint">
+            <command_interface name="effort"/>
+            <state_interface name="position"/>
+            <state_interface name="velocity"/>
+        </joint>
+        <joint name="rf_hip_joint">
+            <command_interface name="effort"/>
+            <state_interface name="position"/>
+            <state_interface name="velocity"/>
+        </joint>
+        <joint name="rf_upper_leg_joint">
+            <command_interface name="effort"/>
+            <state_interface name="position"/>
+            <state_interface name="velocity"/>
+        </joint>
+        <joint name="rf_lower_leg_joint">
+            <command_interface name="effort"/>
+            <state_interface name="position"/>
+            <state_interface name="velocity"/>
+        </joint>
+        <joint name="lh_hip_joint">
+            <command_interface name="effort"/>
+            <state_interface name="position"/>
+            <state_interface name="velocity"/>
+        </joint>
+        <joint name="lh_upper_leg_joint">
+            <command_interface name="effort"/>
+            <state_interface name="position"/>
+            <state_interface name="velocity"/>
+        </joint>
+        <joint name="lh_lower_leg_joint">
+            <command_interface name="effort"/>
+            <state_interface name="position"/>
+            <state_interface name="velocity"/>
+        </joint>
+        <joint name="rh_hip_joint">
+            <command_interface name="effort"/>
+            <state_interface name="position"/>
+            <state_interface name="velocity"/>
+        </joint>
+        <joint name="rh_upper_leg_joint">
+            <command_interface name="effort"/>
+            <state_interface name="position"/>
+            <state_interface name="velocity"/>
+        </joint>
+        <joint name="rh_lower_leg_joint">
+            <command_interface name="effort"/>
+            <state_interface name="position"/>
+            <state_interface name="velocity"/>
+        </joint>
+    </ros2_control>
 </robot>
